File: pcb/upp10a3v1.1.kicad_pcb (KiCad board)
At the start: 2 copper layers, 70 x 61 mm, 15 parts, among them J1 Screw_Terminal_01x06, J2 Screw_Terminal_01x02, J3 IDC26, U1 PCF8574, U2 PCF8574, U3 7407, U4 7407, U5 7407

Commit message: PCB project cont. Gerber files generated;
Parts:
- added C2: 100n, Capacitor_SMD:C_1206_3216Metric_Pad1.33x1.80mm_HandSolder, B.Cu at (70.2, 100.8)
- added C3: 100n, Capacitor_SMD:C_1206_3216Metric_Pad1.33x1.80mm_HandSolder, B.Cu at (69.6, 124.2)
- added C4: 100n, Capacitor_SMD:C_1206_3216Metric_Pad1.33x1.80mm_HandSolder, B.Cu at (71.5, 80.8)
- added C5: 100n, Capacitor_SMD:C_1206_3216Metric_Pad1.33x1.80mm_HandSolder, B.Cu at (81.9, 98.0)
- added C6: 100n, Capacitor_SMD:C_1206_3216Metric_Pad1.33x1.80mm_HandSolder, B.Cu at (81.9, 117.1)
- added C7: 100n, Capacitor_SMD:C_1206_3216Metric_Pad1.33x1.80mm_HandSolder, B.Cu at (106.0, 79.7)
- added C8: 100n, Capacitor_SMD:C_1206_3216Metric_Pad1.33x1.80mm_HandSolder, B.Cu at (98.4, 131.7)
- moved R1 7.85 mm to (60.1, 100.6), turned to 0 degrees
- moved R2 2.05 mm to (63.1, 103.5), turned to 0 degrees
Connections:
- RN1 pad 10: unconnected-(RN1-R9-Pad10) -> Net-(RN1-R9)
- RN1 pad 4: unconnected-(RN1-R3-Pad4) -> Net-(RN1-R3)
- RN1 pad 5: unconnected-(RN1-R4-Pad5) -> Net-(RN1-R4)
- RN1 pad 6: unconnected-(RN1-R5-Pad6) -> Net-(RN1-R5)
- RN1 pad 7: unconnected-(RN1-R6-Pad7) -> Net-(RN1-R6)
- RN1 pad 8: unconnected-(RN1-R7-Pad8) -> Net-(RN1-R7)
- RN1 pad 9: unconnected-(RN1-R8-Pad9) -> Net-(RN1-R8)
- RN2 pad 10: unconnected-(RN2-R9-Pad10) -> /DAC06
- RN2 pad 9: unconnected-(RN2-R8-Pad9) -> /DAC05
- RN3 pad 10: unconnected-(RN3-R9-Pad10) -> /DAC07
- RN3 pad 4: unconnected-(RN3-R3-Pad4) -> /~{WR}
- RN3 pad 5: unconnected-(RN3-R4-Pad5) -> /DAC00
- RN3 pad 6: unconnected-(RN3-R5-Pad6) -> /DAC11
- RN3 pad 7: unconnected-(RN3-R6-Pad7) -> /DAC10
- RN3 pad 8: unconnected-(RN3-R7-Pad8) -> /DAC09
- RN3 pad 9: unconnected-(RN3-R8-Pad9) -> /DAC08
- U1 pad 10: unconnected-(U1-P5-Pad10) -> Net-(RN1-R8)
- U1 pad 11: unconnected-(U1-P6-Pad11) -> Net-(RN1-R7)
- U1 pad 12: unconnected-(U1-P7-Pad12) -> Net-(RN1-R6)
- U1 pad 5: unconnected-(U1-P1-Pad5) -> Net-(RN1-R3)
- U1 pad 6: unconnected-(U1-P2-Pad6) -> Net-(RN1-R4)
- U1 pad 7: unconnected-(U1-P3-Pad7) -> Net-(RN1-R5)
- U1 pad 9: unconnected-(U1-P4-Pad9) -> Net-(RN1-R9)
- U3 pad 1: unconnected-(U3-Pad1) -> Net-(RN1-R8)
- U3 pad 10: unconnected-(U3-Pad10) -> /DAC05
- U3 pad 12: /DAC01 -> /DAC02
- U3 pad 2: unconnected-(U3-Pad2) -> /DAC07
- U3 pad 3: unconnected-(U3-Pad3) -> Net-(RN1-R7)
- U3 pad 4: unconnected-(U3-Pad4) -> /DAC08
- U3 pad 5: unconnected-(U3-Pad5) -> Net-(RN1-R6)
- U3 pad 6: unconnected-(U3-Pad6) -> /DAC09
- U3 pad 8: unconnected-(U3-Pad8) -> /DAC06
- U3 pad 9: unconnected-(U3-Pad9) -> Net-(RN1-R9)
- U4 pad 1: unconnected-(U4-Pad1) -> /GND
- U4 pad 10: unconnected-(U4-Pad10) -> /DAC11
- U4 pad 11: unconnected-(U4-Pad11) -> Net-(RN1-R4)
- U4 pad 12: unconnected-(U4-Pad12) -> /DAC10
- U4 pad 13: unconnected-(U4-Pad13) -> Net-(RN1-R5)
- U4 pad 3: unconnected-(U4-Pad3) -> /GND
- U4 pad 6: unconnected-(U4-Pad6) -> /~{WR}
- U4 pad 8: unconnected-(U4-Pad8) -> /DAC00
- U4 pad 9: unconnected-(U4-Pad9) -> Net-(RN1-R3)
- U5 pad 2: /DAC02 -> /DAC01
Routing:
- net /GND: track 204.9 -> 392.7 mm, vias 3 -> 42
- net /+5V: track 43.9 -> 148.3 mm, vias 1 -> 8
- net Net-(J1-Pin_2): track 0.00 -> 43.1 mm
- net Net-(J1-Pin_3): track 13.0 -> 52.1 mm, vias 2 -> 3
- net Net-(RN1-R9): track 0.00 -> 37.8 mm
- net Net-(J1-Pin_4): track 12.5 -> 49.3 mm, vias 2 -> 3
- net /~{WR}: track 0.00 -> 36.8 mm, vias 0 -> 1
- net /DAC11: track 0.00 -> 35.5 mm
- net /DAC00: track 0.00 -> 33.4 mm
- net Net-(RN5-R8): track 0.00 -> 30.7 mm
- net Net-(RN1-R3): track 0.00 -> 30.6 mm
- net /DAC07: track 0.00 -> 29.8 mm
- net Net-(RN1-R6): track 0.00 -> 29.6 mm
- net /DAC10: track 0.00 -> 28.0 mm
- net Net-(RN1-R4): track 0.00 -> 27.7 mm
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- added copper zone on B.Cu, net /GND
- added copper zone on F.Cu, net /GND

Commit message: Some corrections made;
Parts:
- U1, U2: footprint Package_SO:SOP-16_3.9x9.9mm_P1.27mm -> Package_SO:SOIC-16W_7.5x10.3mm_P1.27mm
- moved C3 3.07 mm to (69.6, 127.3)
Routing:
- net Net-(J1-Pin_3): track 52.1 -> 55.5 mm
- net Net-(J1-Pin_4): track 49.3 -> 52.7 mm
- net /+5V: track 148.3 -> 151.1 mm
- net Net-(RN1-R6): track 29.6 -> 31.6 mm
- net Net-(J1-Pin_2): track 43.1 -> 45.1 mm
- net /GND: track 392.7 -> 394.3 mm, vias 42 -> 43
- net Net-(RN5-R3): track 34.4 -> 35.9 mm
- net Net-(RN5-R6): track 19.2 -> 20.1 mm
- net Net-(RN5-R5): track 24.9 -> 25.8 mm
- net Net-(RN1-R9): track 37.8 -> 37.1 mm
- net Net-(RN5-R1): track 26.6 -> 27.3 mm
- net Net-(RN5-R2): track 29.7 -> 30.4 mm
- net Net-(RN5-R4): track 29.7 -> 30.3 mm
Other:
- board text added: "upp10a3 2025.09.15"
