File: pcb/upp10a3v1.1.kicad_sch (KiCad schematic)
At the start: 15 parts, among them J1 Screw_Terminal_01x06, J2 Screw_Terminal_01x02, J3 IDC26, U1 PCF8574, U2 PCF8574, U3 7407, U4 7407, U5 7407

Commit message: PCB project cont. Gerber files generated;
Parts:
- added C2, C3, C4, C5, C6, C7, C8: 100n, Capacitor_SMD:C_1206_3216Metric_Pad1.33x1.80mm_HandSolder, symbol Device:C
Connections:
- net +15V: now also C7.1, C8.1
- net +5V: now also C2.1, C3.1, C4.1, C5.1, C6.1
- net DAC00: now also RN3.5 (R4), U4.8
- net DAC01: now also U5.2; no longer U3.12
- net DAC02: now also U3.12; no longer U5.2
- net DAC05: now also RN2.9 (R8), U3.10
- net DAC06: now also RN2.10 (R9), U3.8
- net DAC07: now also RN3.10 (R9), U3.2
- net DAC08: now also RN3.9 (R8), U3.4
- net DAC09: now also RN3.8 (R7), U3.6
- net DAC10: now also RN3.7 (R6), U4.12
- net DAC11: now also RN3.6 (R5), U4.10
- net GND: now also U4.1, U4.3, C2.2, C3.2, C4.2, C5.2, C6.2, C7.2, C8.2
- net ~{WR}: now also RN3.4 (R3), U4.6
- net at U4.13: now also RN1.6 (R5), U1.7 (P3)
- net at U4.11: now also RN1.5 (R4), U1.6 (P2)
- net at U3.1: now also RN1.9 (R8), U1.10 (P5)
- net at U3.5: now also RN1.7 (R6), U1.12 (P7)
- net at U1.11 (P6): now also RN1.8 (R7), U3.3
- net at U1.5 (P1): now also RN1.4 (R3), U4.9
- net at U1.9 (P4): now also RN1.10 (R9), U3.9
Other:
- moved on the sheet: C1

Commit message: Some corrections made;
Parts:
- U1, U2: footprint Package_SO:SOP-16_3.9x9.9mm_P1.27mm -> Package_SO:SOIC-16W_7.5x10.3mm_P1.27mm
Changed lines of the file:
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@@
       (effects (font (size 1.27 1.27)) (justify left))
     )
-    (property "Footprint" "Package_SO:SOP-16_3.9x9.9mm_P1.27mm" (at 101.6 50.8 0)
+    (property "Footprint" "Package_SO:SOIC-16W_7.5x10.3mm_P1.27mm" (at 101.6 50.8 0)
       (effects (font (size 1.27 1.27)) hide)
     )
@@
       (effects (font (size 1.27 1.27)) (justify left))
     )
-    (property "Footprint" "Package_SO:SOP-16_3.9x9.9mm_P1.27mm" (at 101.6 185.42 0)
+    (property "Footprint" "Package_SO:SOIC-16W_7.5x10.3mm_P1.27mm" (at 101.6 185.42 0)
       (effects (font (size 1.27 1.27)) hide)
     )
