File: upp10A_pico/upp10A_pico.kicad_pcb (KiCad board)
At the start: 2 copper layers, 111.8 x 66 mm, 74 parts, among them J10 Conn_01x07, J11 Conn_01x03, J3 Conn_01x03, J4 Conn_01x03, J5 Conn_01x05, J6 Conn_01x05, J7 Conn_01x05, J8 Conn_01x05, J9 Conn_01x03, Q1 BF545A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

Commit message: PCB routing completed;
Parts:
- added C15: C, Capacitor_SMD:C_0805_2012Metric_Pad1.18x1.45mm_HandSolder, F.Cu at (97.0, 96.2)
- moved R9 18.9 mm to (75.7, 92.5)
- moved R27 18.8 mm to (78.7, 92.5)
- moved R29 18.8 mm to (76.7, 78.2)
- moved C12 15.4 mm to (86.2, 77.7)
- moved R17 15.4 mm to (121.4, 95.7), turned to 90 degrees
- moved R7 13.9 mm to (134.1, 75.2), turned to 90 degrees
- moved R16 13.5 mm to (131.6, 95.7), turned to 90 degrees
- moved R28 13.3 mm to (76.7, 75.2)
- moved R18 11.4 mm to (129.0, 75.2), turned to 90 degrees
- moved R8 11.1 mm to (131.6, 75.2)
- moved C6 10.0 mm to (95.0, 80.0), turned to 180 degrees
- moved R15 10.00 mm to (128.3, 95.7), turned to 90 degrees
- moved Q7 9.86 mm to (32.6, 105.2)
- moved R19 9.00 mm to (124.0, 75.2), turned to -90 degrees
- moved R6 8.58 mm to (126.5, 75.2)
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Routing:
- net GNDREF: track 0.00 -> 685.1 mm, vias 0 -> 87
- net +15V: track 0.00 -> 138.1 mm, vias 0 -> 3
- net +5V: track 0.00 -> 136.5 mm, vias 0 -> 1
- net +8V: track 0.00 -> 99.6 mm, vias 0 -> 4
- net Net-(U2-Y): track 0.00 -> 85.3 mm, vias 0 -> 3
- net -8V: track 0.00 -> 75.3 mm, vias 0 -> 3
- net Net-(D4-A): track 0.00 -> 67.3 mm
- net +3V3: track 0.00 -> 53.8 mm, vias 0 -> 4
- net Net-(Q7-G): track 0.00 -> 48.5 mm, vias 0 -> 2
- net Net-(Q3-D): track 0.00 -> 45.9 mm, vias 0 -> 3
- net Net-(Q6-G): track 0.00 -> 44.4 mm, vias 0 -> 3
- net Net-(Q1-S): track 0.00 -> 42.0 mm
- net Net-(J10-Pin_6): track 0.00 -> 41.5 mm
- net Net-(Q5-G): track 0.00 -> 40.5 mm, vias 0 -> 3
- net Net-(J10-Pin_5): track 0.00 -> 39.6 mm
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- added copper zone on B.Cu, net GNDREF
- added copper zone on F.Cu, net GNDREF
Other:
- board text added: "locked"
- board text removed: "I2C"
- board text removed: "POMIAR +24V"
- board text removed: "POMIAR I"
- board text removed: "PWM"
- board text removed: "SPARE"
- board text removed: "STYCZNIK"
- board text removed: "UART0"
- board text removed: "UART1"
- board text removed: "ZASILANIE"

Commit message: Made corrections on PCB; added gerber files; added schematic in pdf;
Parts:
- added J1: Conn_01x01, Connector_Pin:Pin_D1.0mm_L10.0mm, F.Cu at (75.2, 116.1)
- added J12: Conn_01x01, Connector_Pin:Pin_D1.0mm_L10.0mm, F.Cu at (52.3, 72.4)
- added J2: Conn_01x01, Connector_Pin:Pin_D1.0mm_L10.0mm, F.Cu at (75.2, 113.0)
Connections:
- U7 pad 21: unconnected-(U7-Pad21) -> Net-(J12-Pin_1)
- U7 pad 4: unconnected-(U7-Pad4) -> Net-(J1-Pin_1)
- U7 pad 5: unconnected-(U7-Pad5) -> Net-(J2-Pin_1)
Routing:
- net Net-(J1-Pin_1): track 0.00 -> 3.72 mm
- net Net-(J12-Pin_1): track 0.00 -> 3.49 mm
- net unconnected-(U7-Pad21): track 3.28 -> 0.00 mm, vias 1 -> 0
- net unconnected-(U7-Pad4): track 2.96 -> 0.00 mm, vias 1 -> 0
- net unconnected-(U7-Pad5): track 2.87 -> 0.00 mm, vias 1 -> 0
- net Net-(J2-Pin_1): track 0.00 -> 2.79 mm
- net Net-(J4-Pin_3): track 15.3 -> 14.7 mm
- net +8V: track 99.6 -> 100.2 mm
